Commit message: Updated

File: src/edge_robot_description/urdf/model.xacro (robot description, xacro)
@@ -89,8 +89,6 @@
             </geometry>
         </collision>
-        <xacro:inertia_lidar/>   <!-- FIX: added missing inertial block -->
-    </link>
-    <!-- Lidar joint: body top is at height above base_link origin.
-         Visual is offset +0.05 inside lidar_link (cylinder sits on top of body). -->
+        <xacro:inertia_lidar/>
+    </link>
     <joint name="lidar_joint" type="fixed">
         <origin xyz="0 0 ${height}" rpy="0 -0.35 0"/>
@@ -109,5 +107,4 @@
             <resolution>1</resolution>
             <min_angle>-3.14159265</min_angle>
-            <!-- FIX #4: Corrected max_angle typo (was 3.141459265, missing '5' digit) -->
             <max_angle>3.14159265</max_angle>
           </horizontal>
